Commit message: Working box detection and track to

File: tennisbot_ws/src/tennisbotmaster/description/robot_core.xacro (robot description, xacro)
@@ -9,7 +9,7 @@
     <xacro:property name="wheel_thickness" value="0.0244"/>
     <xacro:property name="wheel_mass" value="0.05"/>
-    <xacro:property name="wheel_offset_x" value="0.295"/>
-    <xacro:property name="wheel_offset_y" value="0.009"/>
-    <xacro:property name="wheel_offset_z" value="-0.02"/>
+    <xacro:property name="wheel_offset_x" value="0.253"/>
+    <xacro:property name="wheel_offset_y" value="0.003"/>
+    <xacro:property name="wheel_offset_z" value="-0.039"/>
     <xacro:property name="caster_wheel_radius" value="0.0266"/>
     <xacro:property name="caster_wheel_mass" value="0.01"/>
